Commit message: _

File: ros_ws/install/my_robot_description/share/my_robot_description/urdf/mock_components/my_robot_description.ros2_control.xacro (robot description, xacro)
@@ -1 +1,60 @@
-/home/kk/github/ros2_control_moveit_6-dor-arm/ros_ws/src/my_robot_description/urdf/mock_components/my_robot_description.ros2_control.xacro
+<?xml version="1.0"?>
+<robot xmlns:xacro="http://www.ros.org/wiki/xacro">
+    <xacro:macro name="my_robot_description_ros2_control" params="name initial_positions_file">
+        <xacro:property name="initial_positions" value="${xacro.load_yaml(initial_positions_file)['initial_positions']}"/>
+        <ros2_control name="${name}" type="system">
+            <hardware>
+                <plugin>my_robot_hardware_interface/MyRobotHardwareInterface</plugin>
+            </hardware>
+            <joint name="Joint_1">
+                <command_interface name="position"/>
+                <state_interface name="position">
+                  <param name="initial_value">${initial_positions['Joint_1']}</param>
+                </state_interface>
+                <state_interface name="velocity"/>
+            </joint>
+            <joint name="Joint_2">
+                <command_interface name="position"/>
+                <state_interface name="position">
+                  <param name="initial_value">${initial_positions['Joint_2']}</param>
+                </state_interface>
+                <state_interface name="velocity"/>
+            </joint>
+            <joint name="Joint_3">
+                <command_interface name="position"/>
+                <state_interface name="position">
+                  <param name="initial_value">${initial_positions['Joint_3']}</param>
+                </state_interface>
+                <state_interface name="velocity"/>
+            </joint>
+            <joint name="Joint_4">
+                <command_interface name="position"/>
+                <state_interface name="position">
+                  <param name="initial_value">${initial_positions['Joint_4']}</param>
+                </state_interface>
+                <state_interface name="velocity"/>
+            </joint>
+            <joint name="Joint_5">
+                <command_interface name="position"/>
+                <state_interface name="position">
+                  <param name="initial_value">${initial_positions['Joint_5']}</param>
+                </state_interface>
+                <state_interface name="velocity"/>
+            </joint>
+            <joint name="Joint_6">
+                <command_interface name="position"/>
+                <state_interface name="position">
+                  <param name="initial_value">${initial_positions['Joint_6']}</param>
+                </state_interface>
+                <state_interface name="velocity"/>
+            </joint>
+            <joint name="Joint_Gripper">
+                <command_interface name="position"/>
+                <state_interface name="position">
+                  <param name="initial_value">${initial_positions['Joint_Gripper']}</param>
+                </state_interface>
+                <state_interface name="velocity"/>
+            </joint>
+        </ros2_control>
+    </xacro:macro>
+</robot>

File: ros_ws/install/my_robot_description/share/my_robot_description/urdf/mock_components/my_robot_description.urdf.xacro (robot description, xacro)
@@ -1 +1,9 @@
-/home/kk/github/ros2_control_moveit_6-dor-arm/ros_ws/src/my_robot_description/urdf/mock_components/my_robot_description.urdf.xacro
+<?xml version="1.0"?>
+<robot xmlns:xacro="http://www.ros.org/wiki/xacro" name="my_robot_description">
+    <xacro:arg name="initial_positions_file" default="$(find my_robot_moveit_config)/config/initial_positions.yaml" />
+    <!-- Import my_robot_description urdf file -->
+    <xacro:include filename="$(find my_robot_description)/urdf/arm_description.urdf" />
+    <!-- Import control_xacro -->
+    <xacro:include filename="my_robot_description.ros2_control.xacro" />
+    <xacro:my_robot_description_ros2_control name="FakeSystem" initial_positions_file="$(arg initial_positions_file)"/>
+</robot>

File: ros_ws/install/my_robot_moveit_config/share/my_robot_moveit_config/config/my_robot_description.ros2_control.xacro (robot description, xacro)
@@ -1 +1,81 @@
-/home/kk/github/ros2_control_moveit_6-dor-arm/ros_ws/src/my_robot_moveit_config/config/my_robot_description.ros2_control.xacro
+<?xml version="1.0"?>
+<robot xmlns:xacro="http://www.ros.org/wiki/xacro">
+    <xacro:macro name="my_robot_description_ros2_control" params="name initial_positions_file">
+        <xacro:property name="initial_positions" value="${load_yaml(initial_positions_file)['initial_positions']}"/>
+        <ros2_control name="${name}" type="system">
+            <hardware>
+                <plugin>my_robot_hardware_interface/MyRobotHardwareInterface</plugin>
+            </hardware>
+            <joint name="Joint_1">
+                <command_interface name="position">
+                  <param name="min">-3.14</param>
+                  <param name="max">3.14</param>
+                </command_interface>
+                <state_interface name="position">
+                  <param name="initial_value">${initial_positions['Joint_1']}</param>
+                </state_interface>
+                <state_interface name="velocity"/>
+            </joint>
+            <joint name="Joint_2">
+                <command_interface name="position">
+                  <param name="min">-1.57</param>
+                  <param name="max">1.57</param>
+                </command_interface>
+                <state_interface name="position">
+                  <param name="initial_value">${initial_positions['Joint_2']}</param>
+                </state_interface>
+                <state_interface name="velocity"/>
+            </joint>
+            <joint name="Joint_3">
+                <command_interface name="position">
+                  <param name="min">-1.57</param>
+                  <param name="max">1.57</param>
+                </command_interface>
+                <state_interface name="position">
+                  <param name="initial_value">${initial_positions['Joint_3']}</param>
+                </state_interface>
+                <state_interface name="velocity"/>
+            </joint>
+            <joint name="Joint_4">
+                <command_interface name="position">
+                  <param name="min">-1.57</param>
+                  <param name="max">1.57</param>
+                </command_interface>
+                <state_interface name="position">
+                  <param name="initial_value">${initial_positions['Joint_4']}</param>
+                </state_interface>
+                <state_interface name="velocity"/>
+            </joint>
+            <joint name="Joint_5">
+                <command_interface name="position">
+                  <param name="min">-1.46</param>
+                  <param name="max">1.57</param>
+                </command_interface>
+                <state_interface name="position">
+                  <param name="initial_value">${initial_positions['Joint_5']}</param>
+                </state_interface>
+                <state_interface name="velocity"/>
+            </joint>
+            <joint name="Joint_6">
+                <command_interface name="position">
+                  <param name="min">-3.14</param>
+                  <param name="max">3.14</param>
+                </command_interface>
+                <state_interface name="position">
+                  <param name="initial_value">${initial_positions['Joint_6']}</param>
+                </state_interface>
+                <state_interface name="velocity"/>
+            </joint>
+            <joint name="Joint_Gripper">
+                <command_interface name="position">
+                  <param name="min">-0.5</param>
+                  <param name="max">0.18</param>
+                </command_interface>
+                <state_interface name="position">
+                  <param name="initial_value">${initial_positions['Joint_Gripper']}</param>
+                </state_interface>
+                <state_interface name="velocity"/>
+            </joint>
+        </ros2_control>
+    </xacro:macro>
+</robot>

File: ros_ws/install/my_robot_moveit_config/share/my_robot_moveit_config/config/my_robot_description.urdf.xacro (robot description, xacro)
@@ -1 +1,9 @@
-/home/kk/github/ros2_control_moveit_6-dor-arm/ros_ws/src/my_robot_moveit_config/config/my_robot_description.urdf.xacro
+<?xml version="1.0"?>
+<robot xmlns:xacro="http://www.ros.org/wiki/xacro" name="my_robot_description">
+    <xacro:arg name="initial_positions_file" default="initial_positions.yaml" />
+    <!-- Import my_robot_description urdf file -->
+    <xacro:include filename="$(find my_robot_description)/urdf/arm_description.urdf" />
+    <!-- Import control_xacro -->
+    <xacro:include filename="my_robot_description.ros2_control.xacro" />
+    <xacro:my_robot_description_ros2_control name="MyRobotSimulationSystem" initial_positions_file="$(arg initial_positions_file)"/>
+</robot>

File: ros_ws/src/my_robot_moveit_config/config/my_robot_description.ros2_control.xacro (robot description, xacro)
@@ -5,9 +5,11 @@
         <ros2_control name="${name}" type="system">
             <hardware>
-                <!-- By default, set up controllers for simulation. This won't work on real hardware -->
-                <plugin>mock_components/GenericSystem</plugin>
+                <plugin>my_robot_hardware_interface/MyRobotHardwareInterface</plugin>
             </hardware>
             <joint name="Joint_1">
-                <command_interface name="position"/>
+                <command_interface name="position">
+                  <param name="min">-3.14</param>
+                  <param name="max">3.14</param>
+                </command_interface>
                 <state_interface name="position">
                   <param name="initial_value">${initial_positions['Joint_1']}</param>
@@ -16,5 +18,8 @@
             </joint>
             <joint name="Joint_2">
-                <command_interface name="position"/>
+                <command_interface name="position">
+                  <param name="min">-1.57</param>
+                  <param name="max">1.57</param>
+                </command_interface>
                 <state_interface name="position">
                   <param name="initial_value">${initial_positions['Joint_2']}</param>
@@ -23,5 +28,8 @@
             </joint>
             <joint name="Joint_3">
-                <command_interface name="position"/>
+                <command_interface name="position">
+                  <param name="min">-1.57</param>
+                  <param name="max">1.57</param>
+                </command_interface>
                 <state_interface name="position">
                   <param name="initial_value">${initial_positions['Joint_3']}</param>
@@ -30,5 +38,8 @@
             </joint>
             <joint name="Joint_4">
-                <command_interface name="position"/>
+                <command_interface name="position">
+                  <param name="min">-1.57</param>
+                  <param name="max">1.57</param>
+                </command_interface>
                 <state_interface name="position">
                   <param name="initial_value">${initial_positions['Joint_4']}</param>
@@ -37,5 +48,8 @@
             </joint>
             <joint name="Joint_5">
-                <command_interface name="position"/>
+                <command_interface name="position">
+                  <param name="min">-1.46</param>
+                  <param name="max">1.57</param>
+                </command_interface>
                 <state_interface name="position">
                   <param name="initial_value">${initial_positions['Joint_5']}</param>
@@ -44,5 +58,8 @@
             </joint>
             <joint name="Joint_6">
-                <command_interface name="position"/>
+                <command_interface name="position">
+                  <param name="min">-3.14</param>
+                  <param name="max">3.14</param>
+                </command_interface>
                 <state_interface name="position">
                   <param name="initial_value">${initial_positions['Joint_6']}</param>
@@ -51,5 +68,8 @@
             </joint>
             <joint name="Joint_Gripper">
-                <command_interface name="position"/>
+                <command_interface name="position">
+                  <param name="min">-0.5</param>
+                  <param name="max">0.18</param>
+                </command_interface>
                 <state_interface name="position">
                   <param name="initial_value">${initial_positions['Joint_Gripper']}</param>

File: ros_ws/src/my_robot_moveit_config/config/my_robot_description.urdf.xacro (robot description, xacro)
@@ -6,4 +6,4 @@
     <!-- Import control_xacro -->
     <xacro:include filename="my_robot_description.ros2_control.xacro" />
-    <xacro:my_robot_description_ros2_control name="FakeSystem" initial_positions_file="$(arg initial_positions_file)"/>
+    <xacro:my_robot_description_ros2_control name="MyRobotSimulationSystem" initial_positions_file="$(arg initial_positions_file)"/>
 </robot>
